File: Hardware/Matrix_Right.kicad_sch (KiCad schematic)
At the start: 125 parts, among them SW36 PG1350, SW37 PG1350, SW38 PG1350, SW39 PG1350, SW40 PG1350, SW41 PG1350, SW42 PG1350, SW43 PG1350, SW44 PG1350, SW45 PG1350, SW46 PG1350, SW47 PG1350, SW48 PG1350, SW49 PG1350, SW50 PG1350, SW51 PG1350, SW52 PG1350, SW53 PG1350, SW54 PG1350, SW55 PG1350, SW56 PG1350, SW57 PG1350, SW58 PG1350, SW59 PG1350, SW60 PG1350, SW61 PG1350, SW62 PG1350, SW63 PG1350, SW64 PG1350, SW65 PG1350, SW66 ENCODER

Commit message: Pinout and footprints
Updated the MCU footprints because the silkscreen was too close to the edge.
Updated the pinout for the MCUs. The left side seems to be ok, but the right side may need some adjustments.
Connections:
- net COL6_R: no longer SW66.S1
- net GND: now also SW66.S2
- net ENC_SW: no longer names the net of D120.2 (A), SW65.2
- net ENC_SW: no longer SW66.S2
- new net ENC_SW_R: SW66.S1
Other:
- moved on the sheet: D120
Changed lines of the file:
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@@
 		)
 	)
-	(text_box "ENCODER"
+	(text_box "ROTARY ENCODER"
 		(exclude_from_sim no)
 		(at 273.05 22.86 0)
@@
 	)
 	(junction
-		(at 227.33 115.57)
-		(diameter 0)
-		(color 0 0 0 0)
-	)
-	(junction
 		(at 134.62 236.22)
 		(diameter 0)
@@
 	(wire
 		(pts
-			(xy 207.01 120.65) (xy 238.76 120.65)
+			(xy 207.01 120.65) (xy 233.68 120.65)
 		)
 		(stroke
@@
 	(wire
 		(pts
-			(xy 227.33 119.38) (xy 227.33 115.57)
-		)
-		(stroke
-			(width 0)
-			(type default)
-		)
-	)
-	(wire
-		(pts
 			(xy 124.46 237.49) (xy 124.46 236.22)
 		)
@@
 	(wire
 		(pts
-			(xy 238.76 115.57) (xy 238.76 120.65)
+			(xy 233.68 115.57) (xy 233.68 120.65)
 		)
 		(stroke
@@
 	(wire
 		(pts
-			(xy 224.79 119.38) (xy 227.33 119.38)
-		)
-		(stroke
-			(width 0)
-			(type default)
-		)
-	)
-	(wire
-		(pts
 			(xy 229.87 252.73) (xy 243.84 252.73)
 		)
@@
 	(wire
 		(pts
-			(xy 224.79 115.57) (xy 227.33 115.57)
-		)
-		(stroke
-			(width 0)
-			(type default)
-		)
-	)
-	(wire
-		(pts
 			(xy 313.69 71.12) (xy 334.01 71.12)
 		)
@@
 	(wire
 		(pts
+			(xy 364.49 76.2) (xy 364.49 86.36)
+		)
+		(stroke
+			(width 0)
+			(type default)
+		)
+	)
+	(wire
+		(pts
 			(xy 95.25 237.49) (xy 95.25 236.22)
 		)
@@
 	(wire
 		(pts
-			(xy 227.33 115.57) (xy 229.87 115.57)
-		)
-		(stroke
-			(width 0)
-			(type default)
-		)
-	)
-	(wire
-		(pts
 			(xy 92.71 167.64) (xy 106.68 167.64)
 		)
@@
 	(wire
 		(pts
-			(xy 237.49 115.57) (xy 238.76 115.57)
+			(xy 232.41 115.57) (xy 233.68 115.57)
 		)
 		(stroke
@@
 		)
 	)
-	(label "ENC_SW"
-		(at 224.79 119.38 180)
-		(effects
-			(font
-				(size 1.27 1.27)
-			)
-			(justify right bottom)
-		)
-	)
-	(label "ENC_SW"
-		(at 364.49 76.2 0)
-		(effects
-			(font
-				(size 1.27 1.27)
-			)
-			(justify left bottom)
-		)
-	)
 	(global_label "COL4_R"
 		(shape output)
@@
 		)
 	)
-	(global_label "COL6_R"
+	(global_label "ENC_SW_R"
 		(shape output)
 		(at 364.49 71.12 0)
@@
 		)
 		(property "Intersheetrefs" "${INTERSHEET_REFS}"
-			(at 374.5509 71.12 0)
+			(at 377.0908 71.12 0)
 			(hide yes)
 			(show_name no)
@@
 	)
 	(symbol
+		(lib_id "power:GND")
+		(at 364.49 86.36 0)
+		(unit 1)
+		(body_style 1)
+		(exclude_from_sim no)
+		(in_bom yes)
+		(on_board yes)
+		(in_pos_files yes)
+		(dnp no)
+		(fields_autoplaced yes)
+		(property "Reference" "#PWR0253"
+			(at 364.49 92.71 0)
+			(hide yes)
+			(show_name no)
+			(do_not_autoplace no)
+			(effects
+				(font
+					(size 1.27 1.27)
+				)
+			)
+		)
+		(property "Value" "GND"
+			(at 364.49 91.44 0)
+			(show_name no)
+			(do_not_autoplace no)
+			(effects
+				(font
+					(size 1.27 1.27)
+				)
+			)
+		)
+		(property "Footprint" ""
+			(at 364.49 86.36 0)
+			(hide yes)
+			(show_name no)
+			(do_not_autoplace no)
+			(effects
+				(font
+					(size 1.27 1.27)
+				)
+			)
+		)
+		(property "Datasheet" ""
+			(at 364.49 86.36 0)
+			(hide yes)
+			(show_name no)
+			(do_not_autoplace no)
+			(effects
+				(font
+					(size 1.27 1.27)
+				)
+			)
+		)
+		(property "Description" "Power symbol creates a global label with name \"GND\" , ground"
+			(at 364.49 86.36 0)
+			(hide yes)
+			(show_name no)
+			(do_not_autoplace no)
+			(effects
+				(font
+					(size 1.27 1.27)
+				)
+			)
+		)
+		(pin "1"
+		)
+		(instances
+			(project "ValkiriaSplit"
+				(path "/7a2b6783-81dc-46bd-bbde-89342e0b1c5b/9400377e-6428-4a6a-b480-760dc0ea5f15"
+					(reference "#PWR0253")
+					(unit 1)
+				)
+			)
+		)
+	)
+	(symbol
 		(lib_id "Diode:1N4148WT")
 		(at 95.25 85.09 180)
@@
 	(symbol
 		(lib_id "Diode:1N4148WT")
-		(at 233.68 115.57 180)
+		(at 228.6 115.57 180)
 		(unit 1)
 		(body_style 1)
@@
 		(fields_autoplaced yes)
 		(property "Reference" "D120"
-			(at 233.68 109.22 0)
+			(at 228.6 109.22 0)
 			(show_name no)
 			(do_not_autoplace no)
@@
 		)
 		(property "Value" "1N4148WT"
-			(at 233.68 111.76 0)
+			(at 228.6 111.76 0)
 			(show_name no)
 			(do_not_autoplace no)
@@
 		)
 		(property "Footprint" "Diode_SMD:D_SOD-523"
-			(at 233.68 111.125 0)
+			(at 228.6 111.125 0)
 			(hide yes)
 			(show_name no)
@@
 		)
 		(property "Datasheet" "https://www.diodes.com/assets/Datasheets/ds30396.pdf"
-			(at 233.68 115.57 0)
+			(at 228.6 115.57 0)
 			(hide yes)
 			(show_name no)
@@
 		)
 		(property "Description" "75V 0.15A Fast switching Diode, SOD-523"
-			(at 233.68 115.57 0)
+			(at 228.6 115.57 0)
 			(hide yes)
 			(show_name no)
@@
 		)
 		(property "Sim.Device" "D"
-			(at 233.68 115.57 0)
+			(at 228.6 115.57 0)
 			(hide yes)
 			(show_name no)
@@
 		)
 		(property "Sim.Pins" "1=K 2=A"
-			(at 233.68 115.57 0)
+			(at 228.6 115.57 0)
 			(hide yes)
 			(show_name no)
@@
 		)
 		(property "JLC Part" "C7420320"
-			(at 233.68 115.57 0)
+			(at 228.6 115.57 0)
 			(hide yes)
 			(show_name no)
@@
 		)
 		(property "Manufacturer Part" "1N4148WT"
-			(at 233.68 115.57 0)
+			(at 228.6 115.57 0)
 			(hide yes)
 			(show_name no)

Commit message: Reset button and LED switch
Added an LED power switch.
Returned the reset button for bootloader access.
Focus on changing the display to an e-ink one for lower power consumption.
Parts:
- renumbered R27 to R25, R28 to R26, SW36 to SW38, SW37 to SW39, SW38 to SW40, SW39 to SW41, SW40 to SW42, SW41 to SW43, SW42 to SW44, SW43 to SW45, SW44 to SW46, SW45 to SW47, SW46 to SW48, SW47 to SW49, SW48 to SW50, SW49 to SW51, SW50 to SW52, SW51 to SW53, SW52 to SW54, SW53 to SW55, SW54 to SW56, SW55 to SW57, SW56 to SW58, SW57 to SW59, SW58 to SW60, SW59 to SW61, SW60 to SW62, SW61 to SW63, SW62 to SW64, SW63 to SW65, SW64 to SW66, SW65 to SW67, SW66 to SW68
