File: Hardware/ValkiriaSplit.kicad_pcb (KiCad board)
At the start: 2 copper layers, 0 parts

Commit message: Net configurations
Added net labels.
Updated the PCB components.
Parts:
- added C1: 1u, Capacitor_SMD:C_0603_1608Metric, F.Cu at (63.8, 31.5)
- added C10: 4.7u, Capacitor_SMD:C_1206_3216Metric, F.Cu at (379.6, 38.6)
- added C11: 1u, Capacitor_SMD:C_0603_1608Metric, F.Cu at (351.0, 56.0)
- added C12: 1u, Capacitor_SMD:C_0603_1608Metric, F.Cu at (351.0, 58.6)
- added C13: 1u, Capacitor_SMD:C_0603_1608Metric, F.Cu at (122.0, 126.6)
- added C14: 1u, Capacitor_SMD:C_0603_1608Metric, F.Cu at (122.0, 129.1)
- added C15: 1u, Capacitor_SMD:C_0603_1608Metric, F.Cu at (122.0, 131.6)
- added C16: 1u, Capacitor_SMD:C_0603_1608Metric, F.Cu at (122.0, 134.1)
- added C17: 1u, Capacitor_SMD:C_0603_1608Metric, F.Cu at (122.0, 136.6)
- added C18: 1u, Capacitor_SMD:C_0603_1608Metric, F.Cu at (122.0, 139.1)
- added C19: 1u, Capacitor_SMD:C_0603_1608Metric, F.Cu at (122.0, 141.6)
- added C2: 4.7u, Capacitor_SMD:C_1206_3216Metric, F.Cu at (69.8, 60.3)
- added C20: 1u, Capacitor_SMD:C_0603_1608Metric, F.Cu at (126.0, 126.6)
- added C21: 1u, Capacitor_SMD:C_0603_1608Metric, F.Cu at (126.0, 129.1)
- added C22: 1u, Capacitor_SMD:C_0603_1608Metric, F.Cu at (126.0, 131.6)
- added C23: 1u, Capacitor_SMD:C_0603_1608Metric, F.Cu at (126.0, 134.1)
- added C24: 1u, Capacitor_SMD:C_0603_1608Metric, F.Cu at (126.0, 136.6)
- added C25: 1u, Capacitor_SMD:C_0603_1608Metric, F.Cu at (126.0, 139.1)
- added C26: 1u, Capacitor_SMD:C_0603_1608Metric, F.Cu at (126.0, 141.6)
- added C27: 1u, Capacitor_SMD:C_0603_1608Metric, F.Cu at (130.0, 126.6)
- added C28: 1u, Capacitor_SMD:C_0603_1608Metric, F.Cu at (130.0, 129.1)
- added C29: 1u, Capacitor_SMD:C_0603_1608Metric, F.Cu at (130.0, 131.6)
- added C3: 10p, Capacitor_SMD:C_0603_1608Metric, F.Cu at (63.8, 34.0)
- added C30: 1u, Capacitor_SMD:C_0603_1608Metric, F.Cu at (130.0, 134.1)
- added C31: 1u, Capacitor_SMD:C_0603_1608Metric, F.Cu at (130.0, 136.6)
- added C32: 1u, Capacitor_SMD:C_0603_1608Metric, F.Cu at (130.0, 139.1)
- added C33: 1u, Capacitor_SMD:C_0603_1608Metric, F.Cu at (130.0, 141.6)
- added C34: 1u, Capacitor_SMD:C_0603_1608Metric, F.Cu at (134.0, 126.6)
- added C35: 1u, Capacitor_SMD:C_0603_1608Metric, F.Cu at (134.0, 129.1)
- added C36: 1u, Capacitor_SMD:C_0603_1608Metric, F.Cu at (134.0, 131.6)
- added C37: 1u, Capacitor_SMD:C_0603_1608Metric, F.Cu at (134.0, 134.1)
- added C38: 1u, Capacitor_SMD:C_0603_1608Metric, F.Cu at (134.0, 136.6)
- added C39: 1u, Capacitor_SMD:C_0603_1608Metric, F.Cu at (134.0, 139.1)
- added C4: 4.7u, Capacitor_SMD:C_1206_3216Metric, F.Cu at (69.8, 63.7)
- added C40: 1u, Capacitor_SMD:C_0603_1608Metric, F.Cu at (134.0, 141.6)
- added C41: 1u, Capacitor_SMD:C_0603_1608Metric, F.Cu at (138.0, 126.6)
- added C42: 1u, Capacitor_SMD:C_0603_1608Metric, F.Cu at (138.0, 129.1)
- added C43: 1u, Capacitor_SMD:C_0603_1608Metric, F.Cu at (138.0, 131.6)
- added C44: 1u, Capacitor_SMD:C_0603_1608Metric, F.Cu at (138.0, 134.1)
- added C45: 1u, Capacitor_SMD:C_0603_1608Metric, F.Cu at (138.0, 136.6)
- added C46: 1u, Capacitor_SMD:C_0603_1608Metric, F.Cu at (138.0, 139.1)
- added C47: 1u, Capacitor_SMD:C_0603_1608Metric, F.Cu at (138.0, 141.6)
- added C48: 1u, Capacitor_SMD:C_0603_1608Metric, F.Cu at (367.0, 126.6)
- added C49: 1u, Capacitor_SMD:C_0603_1608Metric, F.Cu at (367.0, 129.1)
- added C5: 1u, Capacitor_SMD:C_0603_1608Metric, F.Cu at (63.8, 36.5)
- added C50: 1u, Capacitor_SMD:C_0603_1608Metric, F.Cu at (367.0, 131.6)
- added C51: 1u, Capacitor_SMD:C_0603_1608Metric, F.Cu at (367.0, 134.1)
- added C52: 1u, Capacitor_SMD:C_0603_1608Metric, F.Cu at (367.0, 136.6)
- added C53: 1u, Capacitor_SMD:C_0603_1608Metric, F.Cu at (367.0, 139.1)
- added C54: 1u, Capacitor_SMD:C_0603_1608Metric, F.Cu at (367.0, 141.6)
- added C55: 1u, Capacitor_SMD:C_0603_1608Metric, F.Cu at (371.0, 126.6)
- added C56: 1u, Capacitor_SMD:C_0603_1608Metric, F.Cu at (371.0, 129.1)
- added C57: 1u, Capacitor_SMD:C_0603_1608Metric, F.Cu at (371.0, 131.6)
- added C58: 1u, Capacitor_SMD:C_0603_1608Metric, F.Cu at (371.0, 134.1)
- added C59: 1u, Capacitor_SMD:C_0603_1608Metric, F.Cu at (371.0, 136.6)
- added C6: 1u, Capacitor_SMD:C_0603_1608Metric, F.Cu at (63.8, 39.0)
- added C60: 1u, Capacitor_SMD:C_0603_1608Metric, F.Cu at (371.0, 139.1)
- added C61: 1u, Capacitor_SMD:C_0603_1608Metric, F.Cu at (371.0, 141.6)
- added C62: 1u, Capacitor_SMD:C_0603_1608Metric, F.Cu at (375.0, 126.6)
- added C63: 1u, Capacitor_SMD:C_0603_1608Metric, F.Cu at (375.0, 129.1)
- added C64: 1u, Capacitor_SMD:C_0603_1608Metric, F.Cu at (375.0, 131.6)
- added C65: 1u, Capacitor_SMD:C_0603_1608Metric, F.Cu at (375.0, 134.1)
- added C66: 1u, Capacitor_SMD:C_0603_1608Metric, F.Cu at (375.0, 136.6)
- added C67: 1u, Capacitor_SMD:C_0603_1608Metric, F.Cu at (375.0, 139.1)
- added C68: 1u, Capacitor_SMD:C_0603_1608Metric, F.Cu at (375.0, 141.6)
- added C69: 1u, Capacitor_SMD:C_0603_1608Metric, F.Cu at (379.0, 126.6)
- added C7: 1u, Capacitor_SMD:C_0603_1608Metric, F.Cu at (351.0, 51.0)
- added C70: 1u, Capacitor_SMD:C_0603_1608Metric, F.Cu at (379.0, 129.1)
- added C71: 1u, Capacitor_SMD:C_0603_1608Metric, F.Cu at (379.0, 131.6)
- added C72: 1u, Capacitor_SMD:C_0603_1608Metric, F.Cu at (379.0, 134.1)
- added C73: 1u, Capacitor_SMD:C_0603_1608Metric, F.Cu at (379.0, 136.6)
- added C74: 1u, Capacitor_SMD:C_0603_1608Metric, F.Cu at (379.0, 139.1)
- added C75: 1u, Capacitor_SMD:C_0603_1608Metric, F.Cu at (379.0, 141.6)
- added C76: 1u, Capacitor_SMD:C_0603_1608Metric, F.Cu at (383.0, 126.6)
- added C77: 1u, Capacitor_SMD:C_0603_1608Metric, F.Cu at (383.0, 129.1)
- added C78: 1u, Capacitor_SMD:C_0603_1608Metric, F.Cu at (383.0, 131.6)
- added C79: 1u, Capacitor_SMD:C_0603_1608Metric, F.Cu at (383.0, 134.1)
- added C8: 4.7u, Capacitor_SMD:C_1206_3216Metric, F.Cu at (379.6, 35.3)
- added C80: 1u, Capacitor_SMD:C_0603_1608Metric, F.Cu at (383.0, 136.6)
- added C81: 1u, Capacitor_SMD:C_0603_1608Metric, F.Cu at (383.0, 139.1)
- added C82: 1u, Capacitor_SMD:C_0603_1608Metric, F.Cu at (383.0, 141.6)
- added C9: 10p, Capacitor_SMD:C_0603_1608Metric, F.Cu at (351.0, 53.5)
- added D1: DSK24, Diode_SMD:D_SOD-123F, F.Cu at (64.2, 51.4)
- added D10: SK6812MINI-E, Custom_Parts:LED_SK6812MINI-E_3.2x2.8mm_P1.5mm_ReverseMount, B.Cu at (138.7, 108.3)
- added D100: SK6812MINI-E, Custom_Parts:LED_SK6812MINI-E_3.2x2.8mm_P1.5mm_ReverseMount, B.Cu at (375.3, 122.9)
- added D101: SK6812MINI-E, Custom_Parts:LED_SK6812MINI-E_3.2x2.8mm_P1.5mm_ReverseMount, B.Cu at (366.9, 93.7)
- added D102: 1N4148WT, Diode_SMD:D_SOD-523, F.Cu at (351.3, 154.0)
- added D103: 1N4148WT, Diode_SMD:D_SOD-523, F.Cu at (351.3, 156.4)
- added D104: 1N4148WT, Diode_SMD:D_SOD-523, F.Cu at (351.3, 158.9)
- added D105: 1N4148WT, Diode_SMD:D_SOD-523, F.Cu at (351.3, 161.3)
- added D106: 1N4148WT, Diode_SMD:D_SOD-523, F.Cu at (354.9, 146.6)
- added D107: SK6812MINI-E, Custom_Parts:LED_SK6812MINI-E_3.2x2.8mm_P1.5mm_ReverseMount, B.Cu at (366.9, 98.5)
- added D108: SK6812MINI-E, Custom_Parts:LED_SK6812MINI-E_3.2x2.8mm_P1.5mm_ReverseMount, B.Cu at (366.9, 103.4)
- added D109: SK6812MINI-E, Custom_Parts:LED_SK6812MINI-E_3.2x2.8mm_P1.5mm_ReverseMount, B.Cu at (366.9, 108.3)
- added D11: SK6812MINI-E, Custom_Parts:LED_SK6812MINI-E_3.2x2.8mm_P1.5mm_ReverseMount, B.Cu at (138.7, 113.1)
- added D110: SK6812MINI-E, Custom_Parts:LED_SK6812MINI-E_3.2x2.8mm_P1.5mm_ReverseMount, B.Cu at (366.9, 113.1)
- added D111: SK6812MINI-E, Custom_Parts:LED_SK6812MINI-E_3.2x2.8mm_P1.5mm_ReverseMount, B.Cu at (366.9, 118.0)
- added D112: 1N4148WT, Diode_SMD:D_SOD-523, F.Cu at (354.9, 149.1)
- added D113: 1N4148WT, Diode_SMD:D_SOD-523, F.Cu at (354.9, 151.5)
- added D114: 1N4148WT, Diode_SMD:D_SOD-523, F.Cu at (354.9, 154.0)
- added D115: 1N4148WT, Diode_SMD:D_SOD-523, F.Cu at (354.9, 156.4)
- added D116: 1N4148WT, Diode_SMD:D_SOD-523, F.Cu at (354.9, 158.9)
- added D117: SK6812MINI-E, Custom_Parts:LED_SK6812MINI-E_3.2x2.8mm_P1.5mm_ReverseMount, B.Cu at (366.9, 122.9)
- added D118: SK6812MINI-E, Custom_Parts:LED_SK6812MINI-E_3.2x2.8mm_P1.5mm_ReverseMount, B.Cu at (358.5, 93.7)
- added D119: 1N4148WT, Diode_SMD:D_SOD-523, F.Cu at (354.9, 161.3)
- added D12: 1N4148WT, Diode_SMD:D_SOD-523, F.Cu at (102.7, 146.6)
- added D120: SK6812MINI-E, Custom_Parts:LED_SK6812MINI-E_3.2x2.8mm_P1.5mm_ReverseMount, B.Cu at (358.5, 98.5)
- added D121: SK6812MINI-E, Custom_Parts:LED_SK6812MINI-E_3.2x2.8mm_P1.5mm_ReverseMount, B.Cu at (358.5, 103.4)
- added D122: SK6812MINI-E, Custom_Parts:LED_SK6812MINI-E_3.2x2.8mm_P1.5mm_ReverseMount, B.Cu at (358.5, 108.3)
- added D123: 1N4148WT, Diode_SMD:D_SOD-523, F.Cu at (358.5, 146.6)
- added D124: 1N4148WT, Diode_SMD:D_SOD-523, F.Cu at (358.5, 149.1)
- added D125: 1N4148WT, Diode_SMD:D_SOD-523, F.Cu at (358.5, 151.5)
- added D126: 1N4148WT, Diode_SMD:D_SOD-523, F.Cu at (358.5, 154.0)
- added D127: SK6812MINI-E, Custom_Parts:LED_SK6812MINI-E_3.2x2.8mm_P1.5mm_ReverseMount, B.Cu at (358.5, 113.1)
- added D128: SK6812MINI-E, Custom_Parts:LED_SK6812MINI-E_3.2x2.8mm_P1.5mm_ReverseMount, B.Cu at (358.5, 118.0)
- added D129: 1N4148WT, Diode_SMD:D_SOD-523, F.Cu at (358.5, 156.4)
- added D13: 1N4148WT, Diode_SMD:D_SOD-523, F.Cu at (102.7, 149.1)
- added D130: SK6812MINI-E, Custom_Parts:LED_SK6812MINI-E_3.2x2.8mm_P1.5mm_ReverseMount, B.Cu at (358.5, 122.9)
- added D131: SK6812MINI-E, Custom_Parts:LED_SK6812MINI-E_3.2x2.8mm_P1.5mm_ReverseMount, B.Cu at (350.1, 93.7)
- added D132: SK6812MINI-E, Custom_Parts:LED_SK6812MINI-E_3.2x2.8mm_P1.5mm_ReverseMount, B.Cu at (350.1, 98.5)
- added D133: 1N4148WT, Diode_SMD:D_SOD-523, F.Cu at (358.5, 158.9)
- added D134: 1N4148WT, Diode_SMD:D_SOD-523, F.Cu at (358.5, 161.3)
- added D135: 1N4148WT, Diode_SMD:D_SOD-523, F.Cu at (362.0, 146.6)
- added D136: 1N4148WT, Diode_SMD:D_SOD-523, F.Cu at (362.0, 149.1)
- added D137: SK6812MINI-E, Custom_Parts:LED_SK6812MINI-E_3.2x2.8mm_P1.5mm_ReverseMount, B.Cu at (350.1, 103.4)
- added D138: SK6812MINI-E, Custom_Parts:LED_SK6812MINI-E_3.2x2.8mm_P1.5mm_ReverseMount, B.Cu at (350.1, 108.3)
- added D139: SK6812MINI-E, Custom_Parts:LED_SK6812MINI-E_3.2x2.8mm_P1.5mm_ReverseMount, B.Cu at (350.1, 113.1)
- added D14: 1N4148WT, Diode_SMD:D_SOD-523, F.Cu at (102.7, 151.5)
- added D140: SK6812MINI-E, Custom_Parts:LED_SK6812MINI-E_3.2x2.8mm_P1.5mm_ReverseMount, B.Cu at (350.1, 118.0)
- added D141: SK6812MINI-E, Custom_Parts:LED_SK6812MINI-E_3.2x2.8mm_P1.5mm_ReverseMount, B.Cu at (350.1, 122.9)
- added D142: 1N4148WT, Diode_SMD:D_SOD-523, F.Cu at (362.0, 151.5)
- added D143: 1N4148WT, Diode_SMD:D_SOD-523, F.Cu at (362.0, 154.0)
- added D144: 1N4148WT, Diode_SMD:D_SOD-523, F.Cu at (362.0, 156.4)
- added D145: 1N4148WT, Diode_SMD:D_SOD-523, F.Cu at (362.0, 158.9)
- added D146: 1N4148WT, Diode_SMD:D_SOD-523, F.Cu at (362.0, 161.3)
- added D15: 1N4148WT, Diode_SMD:D_SOD-523, F.Cu at (102.7, 154.0)
- added D16: 1N4148WT, Diode_SMD:D_SOD-523, F.Cu at (102.7, 156.4)
- added D17: SK6812MINI-E, Custom_Parts:LED_SK6812MINI-E_3.2x2.8mm_P1.5mm_ReverseMount, B.Cu at (138.7, 118.0)
- added D18: SK6812MINI-E, Custom_Parts:LED_SK6812MINI-E_3.2x2.8mm_P1.5mm_ReverseMount, B.Cu at (138.7, 122.9)
- added D19: SK6812MINI-E, Custom_Parts:LED_SK6812MINI-E_3.2x2.8mm_P1.5mm_ReverseMount, B.Cu at (130.3, 93.7)
- added D2: DSK24, Diode_SMD:D_SOD-123F, F.Cu at (64.2, 54.8)
- added D20: SK6812MINI-E, Custom_Parts:LED_SK6812MINI-E_3.2x2.8mm_P1.5mm_ReverseMount, B.Cu at (130.3, 98.5)
- added D21: SK6812MINI-E, Custom_Parts:LED_SK6812MINI-E_3.2x2.8mm_P1.5mm_ReverseMount, B.Cu at (130.3, 103.4)
- added D22: 1N4148WT, Diode_SMD:D_SOD-523, F.Cu at (102.7, 158.9)
- added D23: 1N4148WT, Diode_SMD:D_SOD-523, F.Cu at (102.7, 161.3)
- added D24: 1N4148WT, Diode_SMD:D_SOD-523, F.Cu at (106.3, 146.6)
- added D25: 1N4148WT, Diode_SMD:D_SOD-523, F.Cu at (106.3, 149.1)
- added D26: 1N4148WT, Diode_SMD:D_SOD-523, F.Cu at (106.3, 151.5)
- added D27: SK6812MINI-E, Custom_Parts:LED_SK6812MINI-E_3.2x2.8mm_P1.5mm_ReverseMount, B.Cu at (130.3, 108.3)
- added D28: SK6812MINI-E, Custom_Parts:LED_SK6812MINI-E_3.2x2.8mm_P1.5mm_ReverseMount, B.Cu at (130.3, 113.1)
- added D29: SK6812MINI-E, Custom_Parts:LED_SK6812MINI-E_3.2x2.8mm_P1.5mm_ReverseMount, B.Cu at (130.3, 118.0)
- added D3: DSK24, Diode_SMD:D_SOD-123F, F.Cu at (64.2, 58.1)
- added D30: SK6812MINI-E, Custom_Parts:LED_SK6812MINI-E_3.2x2.8mm_P1.5mm_ReverseMount, B.Cu at (130.3, 122.9)
- added D31: SK6812MINI-E, Custom_Parts:LED_SK6812MINI-E_3.2x2.8mm_P1.5mm_ReverseMount, B.Cu at (121.9, 93.7)
- added D32: 1N4148WT, Diode_SMD:D_SOD-523, F.Cu at (106.3, 154.0)
- added D33: 1N4148WT, Diode_SMD:D_SOD-523, F.Cu at (106.3, 156.4)
- added D34: 1N4148WT, Diode_SMD:D_SOD-523, F.Cu at (106.3, 158.9)
- added D35: 1N4148WT, Diode_SMD:D_SOD-523, F.Cu at (106.3, 161.3)
- added D36: 1N4148WT, Diode_SMD:D_SOD-523, F.Cu at (109.9, 146.6)
- added D37: SK6812MINI-E, Custom_Parts:LED_SK6812MINI-E_3.2x2.8mm_P1.5mm_ReverseMount, B.Cu at (121.9, 98.5)
- added D38: SK6812MINI-E, Custom_Parts:LED_SK6812MINI-E_3.2x2.8mm_P1.5mm_ReverseMount, B.Cu at (121.9, 103.4)
- added D39: SK6812MINI-E, Custom_Parts:LED_SK6812MINI-E_3.2x2.8mm_P1.5mm_ReverseMount, B.Cu at (121.9, 108.3)
- added D4: DSK24, Diode_SMD:D_SOD-123F, F.Cu at (374.1, 31.9)
- added D40: SK6812MINI-E, Custom_Parts:LED_SK6812MINI-E_3.2x2.8mm_P1.5mm_ReverseMount, B.Cu at (121.9, 113.1)
- added D41: SK6812MINI-E, Custom_Parts:LED_SK6812MINI-E_3.2x2.8mm_P1.5mm_ReverseMount, B.Cu at (121.9, 118.0)
- added D42: 1N4148WT, Diode_SMD:D_SOD-523, F.Cu at (109.9, 149.1)
- added D43: 1N4148WT, Diode_SMD:D_SOD-523, F.Cu at (109.9, 151.5)
- added D44: 1N4148WT, Diode_SMD:D_SOD-523, F.Cu at (109.9, 154.0)
- added D45: 1N4148WT, Diode_SMD:D_SOD-523, F.Cu at (109.9, 156.4)
- added D46: 1N4148WT, Diode_SMD:D_SOD-523, F.Cu at (109.9, 158.9)
- added D47: SK6812MINI-E, Custom_Parts:LED_SK6812MINI-E_3.2x2.8mm_P1.5mm_ReverseMount, B.Cu at (121.9, 122.9)
- added D48: SK6812MINI-E, Custom_Parts:LED_SK6812MINI-E_3.2x2.8mm_P1.5mm_ReverseMount, B.Cu at (113.5, 93.7)
- added D49: 1N4148WT, Diode_SMD:D_SOD-523, F.Cu at (109.9, 161.3)
- added D5: DSK24, Diode_SMD:D_SOD-123F, F.Cu at (374.1, 35.3)
- added D50: SK6812MINI-E, Custom_Parts:LED_SK6812MINI-E_3.2x2.8mm_P1.5mm_ReverseMount, B.Cu at (113.5, 98.5)
- added D51: SK6812MINI-E, Custom_Parts:LED_SK6812MINI-E_3.2x2.8mm_P1.5mm_ReverseMount, B.Cu at (113.5, 103.4)
- added D52: SK6812MINI-E, Custom_Parts:LED_SK6812MINI-E_3.2x2.8mm_P1.5mm_ReverseMount, B.Cu at (113.5, 108.3)
- added D53: 1N4148WT, Diode_SMD:D_SOD-523, F.Cu at (113.5, 146.6)
- added D54: 1N4148WT, Diode_SMD:D_SOD-523, F.Cu at (113.5, 149.1)
- added D55: 1N4148WT, Diode_SMD:D_SOD-523, F.Cu at (113.5, 151.5)
- added D56: 1N4148WT, Diode_SMD:D_SOD-523, F.Cu at (113.5, 154.0)
- added D57: SK6812MINI-E, Custom_Parts:LED_SK6812MINI-E_3.2x2.8mm_P1.5mm_ReverseMount, B.Cu at (113.5, 113.1)
- added D58: SK6812MINI-E, Custom_Parts:LED_SK6812MINI-E_3.2x2.8mm_P1.5mm_ReverseMount, B.Cu at (113.5, 118.0)
- added D59: 1N4148WT, Diode_SMD:D_SOD-523, F.Cu at (113.5, 156.4)
- added D6: DSK24, Diode_SMD:D_SOD-123F, F.Cu at (374.1, 38.6)
- added D60: SK6812MINI-E, Custom_Parts:LED_SK6812MINI-E_3.2x2.8mm_P1.5mm_ReverseMount, B.Cu at (113.5, 122.9)
- added D61: SK6812MINI-E, Custom_Parts:LED_SK6812MINI-E_3.2x2.8mm_P1.5mm_ReverseMount, B.Cu at (105.1, 93.7)
- added D62: SK6812MINI-E, Custom_Parts:LED_SK6812MINI-E_3.2x2.8mm_P1.5mm_ReverseMount, B.Cu at (105.1, 98.5)
- added D63: 1N4148WT, Diode_SMD:D_SOD-523, F.Cu at (113.5, 158.9)
- added D64: 1N4148WT, Diode_SMD:D_SOD-523, F.Cu at (113.5, 161.3)
- added D65: 1N4148WT, Diode_SMD:D_SOD-523, F.Cu at (117.0, 146.6)
- added D66: 1N4148WT, Diode_SMD:D_SOD-523, F.Cu at (117.0, 149.1)
- added D67: SK6812MINI-E, Custom_Parts:LED_SK6812MINI-E_3.2x2.8mm_P1.5mm_ReverseMount, B.Cu at (105.1, 103.4)
- added D68: SK6812MINI-E, Custom_Parts:LED_SK6812MINI-E_3.2x2.8mm_P1.5mm_ReverseMount, B.Cu at (105.1, 108.3)
- added D69: SK6812MINI-E, Custom_Parts:LED_SK6812MINI-E_3.2x2.8mm_P1.5mm_ReverseMount, B.Cu at (105.1, 113.1)
- added D7: SK6812MINI-E, Custom_Parts:LED_SK6812MINI-E_3.2x2.8mm_P1.5mm_ReverseMount, B.Cu at (138.7, 93.7)
- added D70: SK6812MINI-E, Custom_Parts:LED_SK6812MINI-E_3.2x2.8mm_P1.5mm_ReverseMount, B.Cu at (105.1, 118.0)
- added D71: SK6812MINI-E, Custom_Parts:LED_SK6812MINI-E_3.2x2.8mm_P1.5mm_ReverseMount, B.Cu at (105.1, 122.9)
- added D72: 1N4148WT, Diode_SMD:D_SOD-523, F.Cu at (117.0, 151.5)
- added D73: 1N4148WT, Diode_SMD:D_SOD-523, F.Cu at (117.0, 154.0)
- added D74: 1N4148WT, Diode_SMD:D_SOD-523, F.Cu at (117.0, 156.4)
- added D75: 1N4148WT, Diode_SMD:D_SOD-523, F.Cu at (117.0, 158.9)
- added D76: 1N4148WT, Diode_SMD:D_SOD-523, F.Cu at (117.0, 161.3)
- added D77: SK6812MINI-E, Custom_Parts:LED_SK6812MINI-E_3.2x2.8mm_P1.5mm_ReverseMount, B.Cu at (383.7, 93.7)
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Other:
- board outline added: 375 x 195 mm
- copper layers 2 -> 4

Commit message: Initial layout
Configured the switch and LED initial layout.
Need to add the capacitors for the LEDs and the diodes for the switches.
Parts:
- removed C79, C80, C81, C82: 1u, Capacitor_SMD:C_0603_1608Metric
- removed D145, D146: 1N4148WT, Diode_SMD:D_SOD-523
- added R12: 10K, Resistor_SMD:R_0603_1608Metric, F.Cu at (460.5, 40.4)
- added R3: 10K, Resistor_SMD:R_0603_1608Metric, F.Cu at (-32.6, 39.2)
- added SW69: PG1350, Custom_Parts:PG1350_1.00u_PCB, F.Cu at (262.5, 148.5)
- added SW70: ENCODER, Custom_Parts:ALPS_EC11J_ENCODER, F.Cu at (444.9, 27.2)
- D102, D103, D104, D112, D113, D115, D116, D12, D123, D124, D13, D133, D134, D142, D143, D144, D22, D23, D24, D32, D33, D34, D35, D42, D43, D44, D46, D53, D54, D55, D63, D64, D65, D72, D73, D74, D75, D76, D82, D92, D93: value 1N4148WT -> SK6812MINI-E; footprint Diode_SMD:D_SOD-523 -> Custom_Parts:LED_SK6812MINI-E_3.2x2.8mm_P1.5mm_ReverseMount; moved to B.Cu
- D107, D108, D109, D110, D117, D118, D120, D121, D127, D128, D130, D137, D138, D139, D140, D17, D18, D19, D27, D28, D29, D30, D37, D38, D39, D40, D41, D48, D50, D51, D52, D57, D58, D60, D61, D67, D68, D69, D70, D71, D87, D88, D97, D98, D99: value SK6812MINI-E -> 1N4148WT; footprint Custom_Parts:LED_SK6812MINI-E_3.2x2.8mm_P1.5mm_ReverseMount -> Diode_SMD:D_SOD-523; moved to F.Cu
- SW35, SW68: value ENCODER -> PG1350; footprint Custom_Parts:ALPS_EC11J_ENCODER -> Custom_Parts:PG1350_1.00u_PCB
- SW36: value PG1350 -> ENCODER; footprint Custom_Parts:PG1350_1.00u_PCB -> Custom_Parts:ALPS_EC11J_ENCODER
- moved SW36 342.7 mm to (-48.1, 25.9)
- moved C46 193.1 mm to (326.8, 180.0)
- moved C47 193.1 mm to (326.8, 182.5)
- moved D76 144.6 mm to (260.0, 139.5), turned to 180 degrees
- moved D77 139.7 mm to (260.0, 158.5)
- moved D19 139.4 mm to (32.1, 192.6), turned to 0 degrees
- moved D27 134.3 mm to (32.1, 199.9), turned to 0 degrees
- moved D17 127.4 mm to (32.1, 187.7), turned to 0 degrees
- moved D18 126.1 mm to (32.1, 190.1), turned to 0 degrees
- moved D37 125.8 mm to (35.7, 190.1), turned to 0 degrees
- moved SW51 125.3 mm to (300.6, 67.5)
- moved D133 124.7 mm to (260.0, 82.3), turned to 180 degrees
- moved Q1 124.7 mm to (-55.2, 48.2)
- moved Q2 124.7 mm to (-55.2, 52.7)
- moved D38 124.0 mm to (35.7, 192.6), turned to 0 degrees
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- renumbered R9 to R10, R10 to R11, R11 to R13, R12 to R14, R13 to R15, R14 to R16, R15 to R17, R16 to R18, R3 to R4, R4 to R5, R5 to R6, R6 to R7, R7 to R8, R8 to R9
Connections:
- C46 pad 1: 5VL -> 5VR
- C47 pad 1: 5VL -> 5VR
- D102 pad 1: ROW1_R -> GND
- D102 pad 2: Net-(D102-A) -> Net-(D102-DIN)
- D103 pad 1: ROW2_R -> GND
- D103 pad 2: Net-(D103-A) -> Net-(D103-DIN)
- D104 pad 1: ROW3_R -> GND
- D104 pad 2: Net-(D104-A) -> Net-(D104-DIN)
- D105 pad 1: ROW4_R -> ROW1_R
- D106 pad 1: ROW5_R -> ROW2_R
- D107 pad 1: GND -> ROW3_R
- D107 pad 2: Net-(D107-DIN) -> Net-(D107-A)
- D108 pad 1: GND -> ROW4_R
- D108 pad 2: Net-(D108-DIN) -> Net-(D108-A)
- D109 pad 1: GND -> ROW5_R
- D109 pad 2: Net-(D109-DIN) -> Net-(D109-A)
- D110 pad 1: GND -> ROW6_R
- D110 pad 2: Net-(D100-DOUT) -> Net-(D110-A)
- D111 pad 2: Net-(D101-DOUT) -> Net-(D100-DOUT)
- D112 pad 1: ROW1_R -> GND
- D112 pad 2: Net-(D112-A) -> Net-(D101-DOUT)
- D113 pad 1: ROW2_R -> GND
- D113 pad 2: Net-(D113-A) -> Net-(D102-DOUT)
- D114 pad 1: ROW3_R -> /Matrix_Right/ENC_CW
- D114 pad 2: Net-(D114-A) -> COL4_R
- D115 pad 1: ROW4_R -> GND
- D115 pad 2: Net-(D115-A) -> Net-(D115-DIN)
- D116 pad 1: ROW5_R -> GND
- D116 pad 2: Net-(D116-A) -> Net-(D116-DIN)
- D117 pad 1: GND -> ROW1_R
- D117 pad 2: Net-(D117-DIN) -> Net-(D117-A)
- D118 pad 1: GND -> ROW2_R
- D118 pad 2: Net-(D118-DIN) -> Net-(D118-A)
- D119 pad 1: /Matrix_Right/ENC_CW -> ROW3_R
- D119 pad 2: COL5_R -> Net-(D119-A)
- D12 pad 1: ROW1_L -> GND
- D12 pad 2: Net-(D12-A) -> Net-(D12-DIN)
- D120 pad 1: GND -> ROW4_R
- D120 pad 2: Net-(D109-DOUT) -> Net-(D120-A)
- D121 pad 1: GND -> ROW5_R
- D121 pad 2: Net-(D110-DOUT) -> Net-(D121-A)
- D123 pad 1: ROW1_R -> GND
- D123 pad 2: Net-(D123-A) -> Net-(D112-DOUT)
- D124 pad 1: ROW2_R -> GND
- D124 pad 2: Net-(D124-A) -> Net-(D113-DOUT)
- D125 pad 1: ROW3_R -> /Matrix_Right/ENC_CC
- D125 pad 2: Net-(D125-A) -> COL5_R
- D126 pad 1: ROW4_R -> ROW1_R
- D127 pad 1: GND -> ROW2_R
- D127 pad 2: Net-(D127-DIN) -> Net-(D127-A)
- D128 pad 1: GND -> ROW3_R
- D128 pad 2: Net-(D128-DIN) -> Net-(D128-A)
- D129 pad 1: /Matrix_Right/ENC_CC -> ROW4_R
- D129 pad 2: COL6_R -> Net-(D129-A)
- D13 pad 1: ROW2_L -> GND
- D13 pad 2: Net-(D13-A) -> Net-(D13-DIN)
- D130 pad 1: GND -> ROW5_R
- D130 pad 2: Net-(D120-DOUT) -> Net-(D130-A)
- D131 pad 2: Net-(D121-DOUT) -> Net-(D131-DIN)
- D131 pad 4: Net-(D131-DOUT) -> Net-(D115-DIN)
- D132 pad 2: Net-(D122-DOUT) -> Net-(D132-DIN)
- D132 pad 4: Net-(D132-DOUT) -> Net-(D116-DIN)
- D133 pad 1: ROW1_R -> GND
- D133 pad 2: Net-(D133-A) -> Net-(D122-DOUT)
- D134 pad 1: ROW2_R -> GND
- D134 pad 2: Net-(D134-A) -> Net-(D123-DOUT)
- D135 pad 1: ROW3_R -> ROW1_R
- D136 pad 1: ROW4_R -> ROW2_R
- D137 pad 1: GND -> ROW3_R
- D137 pad 2: Net-(D137-DIN) -> Net-(D137-A)
- D138 pad 1: GND -> ROW4_R
- D138 pad 2: Net-(D138-DIN) -> Net-(D138-A)
- D139 pad 1: GND -> ROW5_R
- D139 pad 2: Net-(D130-DOUT) -> Net-(D139-A)
- D14 pad 1: ROW3_L -> ROW1_L
- D140 pad 1: GND -> ROW6_R
- D140 pad 2: Net-(D131-DOUT) -> /Matrix_Right/ENC_SW
- D141 pad 2: Net-(D132-DOUT) -> Net-(D141-DIN)
- D141 pad 4: unconnected-(D141-DOUT-Pad4) -> Net-(D131-DIN)
- D142 pad 1: ROW1_R -> GND
- D142 pad 2: Net-(D142-A) -> Net-(D142-DIN)
- D143 pad 1: ROW2_R -> GND
- D143 pad 2: Net-(D143-A) -> Net-(D133-DOUT)
- D144 pad 1: ROW3_R -> GND
- D144 pad 2: Net-(D144-A) -> Net-(D134-DOUT)
- D15 pad 1: ROW4_L -> ROW2_L
- D16 pad 1: ROW5_L -> ROW3_L
- D17 pad 1: GND -> ROW4_L
- D17 pad 2: Net-(D17-DIN) -> Net-(D17-A)
- D18 pad 1: GND -> ROW5_L
- D18 pad 2: Net-(D18-DIN) -> Net-(D18-A)
- D19 pad 1: GND -> ROW6_L
- D19 pad 2: Net-(D19-DIN) -> Net-(D19-A)
- D20 pad 2: Net-(D10-DOUT) -> Net-(D20-DIN)
- D21 pad 2: Net-(D11-DOUT) -> Net-(D10-DOUT)
- D22 pad 1: ROW1_L -> GND
- D22 pad 2: Net-(D22-A) -> Net-(D11-DOUT)
- D23 pad 1: ROW2_L -> GND
- D23 pad 2: Net-(D23-A) -> Net-(D23-DIN)
- D24 pad 1: ROW3_L -> GND
- D24 pad 2: Net-(D24-A) -> Net-(D24-DIN)
- D25 pad 1: ROW4_L -> ROW1_L
- D26 pad 1: ROW5_L -> ROW2_L
- D27 pad 1: GND -> ROW3_L
- D27 pad 2: Net-(D27-DIN) -> Net-(D27-A)
- D28 pad 1: GND -> ROW4_L
- D28 pad 2: Net-(D28-DIN) -> Net-(D28-A)
- D29 pad 1: GND -> ROW5_L
- D29 pad 2: Net-(D19-DOUT) -> Net-(D29-A)
- D30 pad 1: GND -> ROW6_L
- D30 pad 2: Net-(D20-DOUT) -> Net-(D30-A)
- D31 pad 2: Net-(D21-DOUT) -> Net-(D20-DOUT)
- D32 pad 1: ROW1_L -> GND
- D32 pad 2: Net-(D32-A) -> Net-(D21-DOUT)
- D33 pad 1: ROW2_L -> GND
- D33 pad 2: Net-(D33-A) -> Net-(D22-DOUT)
- D34 pad 1: ROW3_L -> GND
- D34 pad 2: Net-(D34-A) -> Net-(D34-DIN)
- D35 pad 1: ROW4_L -> GND
- D35 pad 2: Net-(D35-A) -> Net-(D35-DIN)
- D36 pad 1: ROW5_L -> ROW1_L
- D37 pad 1: GND -> ROW2_L
- D37 pad 2: Net-(D37-DIN) -> Net-(D37-A)
- D38 pad 1: GND -> ROW3_L
- D38 pad 2: Net-(D38-DIN) -> Net-(D38-A)
- D39 pad 1: GND -> ROW4_L
- D39 pad 2: Net-(D29-DOUT) -> Net-(D39-A)
- D40 pad 1: GND -> ROW5_L
- D40 pad 2: Net-(D30-DOUT) -> Net-(D40-A)
- D41 pad 1: GND -> ROW6_L
- D41 pad 2: Net-(D31-DOUT) -> Net-(D41-A)
- D42 pad 1: ROW1_L -> GND
- D42 pad 2: Net-(D42-A) -> Net-(D31-DOUT)
- D43 pad 1: ROW2_L -> GND
- D43 pad 2: Net-(D43-A) -> Net-(D32-DOUT)
- D44 pad 1: ROW3_L -> GND
- D44 pad 2: Net-(D44-A) -> Net-(D33-DOUT)
- D45 pad 1: ROW4_L -> /Matrix_Left/ENC_CW
- D45 pad 2: Net-(D45-A) -> COL4_L
- D46 pad 1: ROW5_L -> GND
- D46 pad 2: Net-(D46-A) -> Net-(D46-DIN)
- D47 pad 4: Net-(D37-DIN) -> Net-(D35-DIN)
- D48 pad 1: GND -> ROW1_L
- D48 pad 2: Net-(D48-DIN) -> Net-(D48-A)
- D49 pad 1: /Matrix_Left/ENC_CW -> ROW2_L
- D49 pad 2: COL5_L -> Net-(D49-A)
- D50 pad 1: GND -> ROW3_L
- D50 pad 2: Net-(D39-DOUT) -> Net-(D50-A)
- D51 pad 1: GND -> ROW4_L
- D51 pad 2: Net-(D40-DOUT) -> Net-(D51-A)
- D52 pad 1: GND -> ROW5_L
- D52 pad 2: Net-(D41-DOUT) -> Net-(D52-A)
- D53 pad 1: ROW1_L -> GND
- D53 pad 2: Net-(D53-A) -> Net-(D42-DOUT)
- D54 pad 1: ROW2_L -> GND
- D54 pad 2: Net-(D54-A) -> Net-(D43-DOUT)
- D55 pad 1: ROW3_L -> GND
- D55 pad 2: Net-(D55-A) -> Net-(D44-DOUT)
- D56 pad 1: ROW4_L -> /Matrix_Left/ENC_CC
- D56 pad 2: Net-(D56-A) -> COL5_L
- D57 pad 1: GND -> ROW1_L
- D57 pad 2: Net-(D57-DIN) -> Net-(D57-A)
- D58 pad 1: GND -> ROW2_L
- D58 pad 2: Net-(D58-DIN) -> Net-(D58-A)
- D59 pad 1: /Matrix_Left/ENC_CC -> ROW3_L
- D59 pad 2: COL6_L -> Net-(D59-A)
- D60 pad 1: GND -> ROW4_L
- D60 pad 2: Net-(D50-DOUT) -> Net-(D60-A)
- D61 pad 1: GND -> ROW5_L
- D61 pad 2: Net-(D51-DOUT) -> Net-(D61-A)
- D62 pad 2: Net-(D52-DOUT) -> Net-(D62-DIN)
- D62 pad 4: Net-(D62-DOUT) -> Net-(D46-DIN)
- D63 pad 1: ROW1_L -> GND
- D63 pad 2: Net-(D63-A) -> Net-(D63-DIN)
- D64 pad 1: ROW2_L -> GND
- D64 pad 2: Net-(D64-A) -> Net-(D53-DOUT)
- D65 pad 1: ROW3_L -> GND
- D65 pad 2: Net-(D65-A) -> Net-(D54-DOUT)
- D66 pad 1: ROW4_L -> ROW1_L
- D67 pad 1: GND -> ROW2_L
- D67 pad 2: Net-(D67-DIN) -> Net-(D67-A)
- D68 pad 1: GND -> ROW3_L
- D68 pad 2: Net-(D68-DIN) -> Net-(D68-A)
- D69 pad 1: GND -> ROW4_L
- D69 pad 2: Net-(D60-DOUT) -> Net-(D69-A)
- D7 pad 2: Net-(D17-DOUT) -> Net-(D12-DOUT)
- D70 pad 1: GND -> ROW5_L
- D70 pad 2: Net-(D61-DOUT) -> Net-(D70-A)
- D71 pad 1: GND -> ROW6_L
- D71 pad 2: Net-(D62-DOUT) -> /Matrix_Left/ENC_SW
- D72 pad 1: ROW1_L -> GND
- D72 pad 2: Net-(D72-A) -> Net-(D72-DIN)
- D73 pad 1: ROW2_L -> GND
- D73 pad 2: Net-(D73-A) -> Net-(D73-DIN)
- D74 pad 1: ROW3_L -> GND
- D74 pad 2: Net-(D74-A) -> Net-(D64-DOUT)
- D75 pad 1: ROW4_L -> GND
- D75 pad 2: Net-(D75-A) -> Net-(D65-DOUT)
- D76 pad 1: ROW5_L -> GND
- D76 pad 2: /Matrix_Left/ENC_SW -> Net-(D76-DIN)
- D78 pad 2: Net-(D78-DIN) -> LED_DATA_R
- D79 pad 2: LED_DATA_R -> Net-(D76-DOUT)
- D8 pad 2: Net-(D18-DOUT) -> Net-(D13-DOUT)
- D81 pad 2: Net-(D78-DOUT) -> Net-(D81-DIN)
- D81 pad 4: Net-(D81-DOUT) -> Net-(D76-DIN)
- D82 pad 1: ROW1_R -> GND
- D82 pad 2: Net-(D82-A) -> Net-(D82-DIN)
- D83 pad 1: ROW2_R -> ROW1_R
- D84 pad 1: ROW3_R -> ROW2_R
- D85 pad 1: ROW4_R -> ROW3_R
- D86 pad 1: ROW5_R -> ROW4_R
- D87 pad 1: GND -> ROW5_R
- D87 pad 2: Net-(D87-DIN) -> Net-(D87-A)
- D88 pad 1: GND -> ROW6_R
- D88 pad 2: Net-(D88-DIN) -> Net-(D88-A)
- D89 pad 2: Net-(D79-DOUT) -> Net-(D78-DOUT)
- D89 pad 4: Net-(D89-DOUT) -> Net-(D100-DIN)
- D9 pad 4: Net-(D19-DIN) -> Net-(D20-DIN)
- D90 pad 2: Net-(D80-DOUT) -> Net-(D79-DOUT)
- D90 pad 4: Net-(D100-DIN) -> Net-(D101-DIN)
- D91 pad 2: Net-(D81-DOUT) -> Net-(D80-DOUT)
- D91 pad 4: Net-(D101-DIN) -> Net-(D102-DIN)
- D92 pad 1: ROW1_R -> GND
- D92 pad 2: Net-(D92-A) -> Net-(D103-DOUT)
- D93 pad 1: ROW2_R -> GND
- D93 pad 2: Net-(D93-A) -> Net-(D104-DOUT)
- D94 pad 1: ROW3_R -> ROW1_R
- D95 pad 1: ROW4_R -> ROW2_R
- D96 pad 1: ROW5_R -> ROW3_R
- D97 pad 1: GND -> ROW4_R
- D97 pad 2: Net-(D107-DOUT) -> Net-(D97-A)
- D98 pad 1: GND -> ROW5_R
- D98 pad 2: Net-(D108-DOUT) -> Net-(D98-A)
- D99 pad 1: GND -> ROW6_R
- D99 pad 2: Net-(D89-DOUT) -> Net-(D99-A)
- SW10 pad 2: Net-(D24-A) -> Net-(D26-A)
- SW11 pad 2: Net-(D25-A) -> Net-(D27-A)
- SW12 pad 2: Net-(D26-A) -> Net-(D28-A)
- SW13 pad 1: COL3_L -> COL2_L
- SW13 pad 2: Net-(D32-A) -> Net-(D29-A)
- SW14 pad 1: COL3_L -> COL2_L
- SW14 pad 2: Net-(D33-A) -> Net-(D30-A)
- SW15 pad 2: Net-(D34-A) -> Net-(D36-A)
- SW16 pad 2: Net-(D35-A) -> Net-(D37-A)
- SW17 pad 2: Net-(D36-A) -> Net-(D38-A)
- SW18 pad 1: COL4_L -> COL3_L
- SW18 pad 2: Net-(D42-A) -> Net-(D39-A)
- SW19 pad 1: COL4_L -> COL3_L
- SW19 pad 2: Net-(D43-A) -> Net-(D40-A)
- SW20 pad 1: COL4_L -> COL3_L
- SW20 pad 2: Net-(D44-A) -> Net-(D41-A)
- SW21 pad 2: Net-(D45-A) -> Net-(D48-A)
- SW22 pad 2: Net-(D46-A) -> Net-(D49-A)
- SW23 pad 1: COL5_L -> COL4_L
- SW23 pad 2: Net-(D53-A) -> Net-(D50-A)
- SW24 pad 1: COL5_L -> COL4_L
- SW24 pad 2: Net-(D54-A) -> Net-(D51-A)
- SW25 pad 1: COL5_L -> COL4_L
- SW25 pad 2: Net-(D55-A) -> Net-(D52-A)
- SW26 pad 2: Net-(D56-A) -> Net-(D57-A)
- SW27 pad 1: COL6_L -> COL5_L
- SW27 pad 2: Net-(D63-A) -> Net-(D58-A)
- SW28 pad 1: COL6_L -> COL5_L
- SW28 pad 2: Net-(D64-A) -> Net-(D59-A)
- SW29 pad 1: COL6_L -> COL5_L
- SW29 pad 2: Net-(D65-A) -> Net-(D60-A)
- SW3 pad 2: Net-(D12-A) -> Net-(D14-A)
- SW30 pad 1: COL6_L -> COL5_L
- SW30 pad 2: Net-(D66-A) -> Net-(D61-A)
- SW31 pad 1: COL7_L -> COL6_L
- SW31 pad 2: Net-(D72-A) -> Net-(D66-A)
- SW32 pad 1: COL7_L -> COL6_L
- SW32 pad 2: Net-(D73-A) -> Net-(D67-A)
- SW33 pad 1: COL7_L -> COL6_L
- SW33 pad 2: Net-(D74-A) -> Net-(D68-A)
- SW34 pad 1: COL7_L -> COL6_L
- SW34 pad 2: Net-(D75-A) -> Net-(D69-A)
- SW4 pad 2: Net-(D13-A) -> Net-(D15-A)
- SW41 pad 1: COL2_R -> COL1_R
- SW41 pad 2: Net-(D92-A) -> Net-(D87-A)
- SW42 pad 1: COL2_R -> COL1_R
- SW42 pad 2: Net-(D93-A) -> Net-(D88-A)
- SW46 pad 1: COL3_R -> COL2_R
- SW46 pad 2: Net-(D102-A) -> Net-(D97-A)
- SW47 pad 1: COL3_R -> COL2_R
- SW47 pad 2: Net-(D103-A) -> Net-(D98-A)
- SW48 pad 1: COL3_R -> COL2_R
- SW48 pad 2: Net-(D104-A) -> Net-(D99-A)
- SW5 pad 2: Net-(D14-A) -> Net-(D16-A)
- SW51 pad 1: COL4_R -> COL3_R
- SW51 pad 2: Net-(D112-A) -> Net-(D107-A)
- SW52 pad 1: COL4_R -> COL3_R
- SW52 pad 2: Net-(D113-A) -> Net-(D108-A)
- SW53 pad 1: COL4_R -> COL3_R
- SW53 pad 2: Net-(D114-A) -> Net-(D109-A)
- SW54 pad 1: COL4_R -> COL3_R
- SW54 pad 2: Net-(D115-A) -> Net-(D110-A)
- SW55 pad 2: Net-(D116-A) -> Net-(D117-A)
- SW56 pad 1: COL5_R -> COL4_R
- SW56 pad 2: Net-(D123-A) -> Net-(D118-A)
- SW57 pad 1: COL5_R -> COL4_R
- SW57 pad 2: Net-(D124-A) -> Net-(D119-A)
- SW58 pad 1: COL5_R -> COL4_R
- SW58 pad 2: Net-(D125-A) -> Net-(D120-A)
- SW59 pad 1: COL5_R -> COL4_R
- SW59 pad 2: Net-(D126-A) -> Net-(D121-A)
- SW6 pad 2: Net-(D15-A) -> Net-(D17-A)
- SW60 pad 1: COL6_R -> COL5_R
- SW60 pad 2: Net-(D133-A) -> Net-(D126-A)
- SW61 pad 1: COL6_R -> COL5_R
- SW61 pad 2: Net-(D134-A) -> Net-(D127-A)
- SW62 pad 1: COL6_R -> COL5_R
- SW62 pad 2: Net-(D135-A) -> Net-(D128-A)
- SW63 pad 1: COL6_R -> COL5_R
- SW63 pad 2: Net-(D136-A) -> Net-(D129-A)
- SW64 pad 1: COL7_R -> COL5_R
- SW64 pad 2: Net-(D142-A) -> Net-(D130-A)
- SW65 pad 1: COL7_R -> COL6_R
- SW65 pad 2: Net-(D143-A) -> Net-(D135-A)
- SW66 pad 1: COL7_R -> COL6_R
- SW66 pad 2: Net-(D144-A) -> Net-(D136-A)
- SW67 pad 1: COL7_R -> COL6_R
- SW67 pad 2: Net-(D145-A) -> Net-(D137-A)
- SW7 pad 2: Net-(D16-A) -> Net-(D18-A)
- SW8 pad 1: COL2_L -> COL1_L
- SW8 pad 2: Net-(D22-A) -> Net-(D19-A)
- SW9 pad 2: Net-(D23-A) -> Net-(D25-A)
- U2 pad 23: /Control_Left/LED_EN -> ROW6_L
- U2 pad 7: COL7_L -> /Control_Left/LED_EN
- U4 pad 23: /Control_Right/LED_EN -> ROW6_R
- U4 pad 7: COL7_R -> /Control_Right/LED_EN
Other:
- board size 375 x 195 mm -> 350 x 195 mm

Commit message: Diode and LED layout
Updated the layout for the LEDs and the diodes.
Need to decide on a final layout for the extra keys and encoders.
Parts:
- C13, C14, C15, C16, C17, C18, C19, C20, C21, C22, C23, C24, C25, C26, C27, C28, C29, C30, C31, C32, C33, C34, C35, C36, C37, C38, C39, C40, C41, C42, C43, C44, C45, C46, C47, C48, C49, C50, C51, C52, C53, C54, C55, C56, C57, C58, C59, C60, C61, C62, C63, C64, C65, C66, C67, C68, C69, C70, C71, C72, C73, C74, C75, C76, C77, C78, D105, D106, D107, D108, D109, D110, D114, D117, D118, D119, D120, D121, D125, D126, D127, D128, D129, D130, D135, D136, D137, D138, D139, D14, D140, D15, D16, D17, D18, D19, D25, D26, D27, D28, D29, D30, D36, D37, D38, D39, D40, D41, D45, D48, D49, D50, D51, D52, D56, D57, D58, D59, D60, D61, D66, D67, D68, D69, D70, D71, D83, D84, D85, D86, D87, D88, D94, D95, D96, D97, D98, D99: moved to B.Cu
- moved D71 195.9 mm to (-58.1, 32.0), turned to 90 degrees
- moved D56 191.1 mm to (-60.5, 32.0), turned to 90 degrees
- moved D140 181.6 mm to (435.4, 33.3), turned to 90 degrees
- moved D45 180.2 mm to (-63.0, 32.0), turned to 90 degrees
- moved D125 177.6 mm to (433.0, 33.3), turned to 90 degrees
- moved D114 163.3 mm to (430.6, 33.3), turned to 90 degrees
- moved D66 152.5 mm to (148.3, 77.4), turned to 90 degrees
- moved D70 149.8 mm to (129.2, 75.0), turned to 90 degrees
- moved D67 141.0 mm to (148.3, 96.4), turned to 90 degrees
- moved C29 138.9 mm to (141.9, 85.2), turned to 180 degrees
- moved D95 138.5 mm to (287.3, 75.0), turned to 90 degrees
- moved D57 137.1 mm to (129.2, 94.0), turned to 90 degrees
- moved D96 133.1 mm to (268.3, 96.4), turned to 90 degrees
- moved D14 133.0 mm to (110.2, 72.6), turned to 90 degrees
- moved D83 132.7 mm to (268.3, 77.4), turned to 90 degrees
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
Commit message: Layout coordination
Coordinated the layout with the schematic.
Finished the initial switch layout.
Need to decide on a complete layout for the keyboard and assign the auxiliary keys.
Parts:
- removed the C17 at (84.8, 120.9)
- removed the C22 at (122.9, 159.0)
- removed the C27 at (103.8, 80.4)
- removed the C32 at (65.8, 144.7)
- removed the C37 at (141.9, 123.3)
- removed the C50 at (300.1, 99.4)
- removed the C55 at (300.1, 185.1)
- removed the C60 at (338.1, 87.6)
- removed the C65 at (357.2, 144.7)
- removed the C70 at (357.2, 106.6)
- removed the D102 at (336.2, 160.9)
- removed the D11 at (140.0, 182.2)
- removed the D110 at (363.5, 117.9)
- removed the D113 at (279.1, 79.9)
- removed the D114 at (430.6, 33.3)
- removed the D124 at (355.2, 160.9)
- removed D125, D140: 1N4148WT, Diode_SMD:D_SOD-523
- removed the D19 at (53.0, 79.8)
- removed the D22 at (82.8, 79.9)
- removed the D30 at (72.1, 98.8)
- removed the D33 at (63.8, 122.8)
- removed the D41 at (91.1, 132.1)
- removed the D44 at (140.0, 82.3)
- removed the D45 at (-63.0, 32.0)
- removed the D55 at (101.9, 96.6)
- removed the D56 at (-60.5, 32.0)
- removed the D71 at (-58.1, 32.0)
- removed the D80 at (298.1, 134.7)
- removed the D88 at (287.3, 151.2)
- removed the D91 at (260.0, 120.4)
- removed the D99 at (325.4, 132.1)
- removed the SW14 at (66.3, 93.7)
- removed the SW20 at (85.4, 127.0)
- removed the SW35 at (123.5, 69.9)
- removed the SW42 at (281.6, 146.1)
- removed the SW48 at (319.7, 127.0)
- removed the SW54 at (357.8, 112.8)
- removed SW69: PG1350, Custom_Parts:PG1350_1.00u_PCB
- removed the SW8 at (47.3, 74.7)
- added C13: 1u, Capacitor_SMD:C_0603_1608Metric, F.Cu at (141.9, 123.3)
- added C42: 100n, Capacitor_SMD:C_0603_1608Metric, F.Cu at (-26.8, 144.0)
- added C43: 100n, Capacitor_SMD:C_0603_1608Metric, F.Cu at (-26.8, 146.5)
- added C44: 1u, Capacitor_SMD:C_0603_1608Metric, B.Cu at (357.2, 144.7)
- added C73: 100n, Capacitor_SMD:C_0603_1608Metric, F.Cu at (451.9, 147.7)
- added C74: 100n, Capacitor_SMD:C_0603_1608Metric, F.Cu at (451.9, 150.2)
- added D66: SK6812MINI-E, Custom_Parts:LED_SK6812MINI-E_3.2x2.8mm_P1.5mm_ReverseMount, B.Cu at (279.1, 79.9)
- added D7: SK6812MINI-E, Custom_Parts:LED_SK6812MINI-E_3.2x2.8mm_P1.5mm_ReverseMount, B.Cu at (63.8, 122.8)
- added FID1: Fiducial, Fiducial:Fiducial_1mm_Mask2mm, F.Cu at (196.0, 242.2)
- added FID2: Fiducial, Fiducial:Fiducial_1mm_Mask2mm, F.Cu at (196.0, 245.8)
- added FID3: Fiducial, Fiducial:Fiducial_1mm_Mask2mm, F.Cu at (196.0, 249.3)
- added FID4: Fiducial, Fiducial:Fiducial_1mm_Mask2mm, F.Cu at (196.0, 252.8)
- added H1: MountingHole, MountingHole:ToolingHole_1.152mm, F.Cu at (199.0, 241.7)
- added H2: MountingHole, MountingHole:ToolingHole_1.152mm, F.Cu at (199.0, 244.1)
- added H3: MountingHole, MountingHole:ToolingHole_1.152mm, F.Cu at (199.0, 246.6)
- added H4: MountingHole, MountingHole:ToolingHole_1.152mm, F.Cu at (199.0, 249.0)
- added R19: 0, Resistor_SMD:R_0603_1608Metric, F.Cu at (-18.8, 141.5)
- added R20: 0, Resistor_SMD:R_0603_1608Metric, F.Cu at (-18.8, 144.0)
- added R21: 0, Resistor_SMD:R_0603_1608Metric, F.Cu at (459.9, 145.2)
- added R22: 0, Resistor_SMD:R_0603_1608Metric, F.Cu at (459.9, 147.7)
- moved D118 180.0 mm to (448.3, 153.2)
- moved D59 176.1 mm to (-30.4, 149.4)
- moved C67 123.4 mm to (357.2, 106.6)
- moved SW8 113.0 mm to (47.3, 74.7)
- moved C45 113.0 mm to (338.1, 87.6)
- moved D21 113.0 mm to (53.0, 79.8)
- moved D28 109.2 mm to (82.8, 79.9)
- moved J5 105.1 mm to (453.9, 154.0)
- moved R13 102.4 mm to (455.9, 145.2)
- moved R11 102.4 mm to (455.9, 140.2)
- moved R12 102.4 mm to (455.9, 142.7)
- moved R14 102.4 mm to (455.9, 147.7)
- moved R15 102.4 mm to (455.9, 150.2)
- moved J2 101.3 mm to (-24.8, 150.3)
- moved R4 100.3 mm to (-22.8, 141.5)
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- renumbered C13 to C14, C14 to C15, C15 to C16, C16 to C17, C23 to C22, C24 to C23, C25 to C24, C26 to C25, C28 to C26, C29 to C27, C30 to C28, C31 to C29, C33 to C30, C34 to C31, C35 to C32, C36 to C33, C38 to C34, C39 to C35, C40 to C36, C41 to C37, C42 to C38, C43 to C39, C44 to C40, C45 to C41, C46 to C45, C47 to C46, C48 to C47, C49 to C48, C51 to C49, C52 to C50, C53 to C51, C54 to C52, C56 to C53, C57 to C54, C58 to C55, C59 to C56, C61 to C57, C62 to C58, C63 to C59, C64 to C60, C66 to C61, C67 to C62, C68 to C63, C69 to C64, C71 to C65, C72 to C66, C73 to C67, C74 to C68, C75 to C69, C76 to C70, C77 to C71, C78 to C72, D9 to D10, D119 to D100, D120 to D101, D121 to D102, D115 to D103, D116 to D104, D122 to D105, D123 to D106, D126 to D107, D127 to D108, D128 to D109, D10 to D11, D129 to D110, D130 to D111, D131 to D112, D132 to D113, D135 to D114, D136 to D115, D137 to D116, D138 to D117, D139 to D118, D133 to D119, D14 to D12, D134 to D120, D141 to D121, D142 to D122, D143 to D123, D144 to D124, D15 to D13, D16 to D14, D17 to D15, D18 to D16, D12 to D17, D13 to D18, D20 to D19, D21 to D20, D25 to D21, D26 to D22, D27 to D23, D28 to D24, D29 to D25, D23 to D26, D24 to D27, D31 to D28, D32 to D29, D36 to D30, D37 to D31, D38 to D32, D39 to D33, D40 to D34, D34 to D35, D35 to D36, D42 to D37, D43 to D38, D48 to D39, D49 to D40, D50 to D41, D51 to D42, D52 to D43, D46 to D44, D47 to D45, D53 to D46, D54 to D47, D57 to D48, D58 to D49, D59 to D50, D60 to D51, D61 to D52, D62 to D53, D63 to D54, D66 to D55, D67 to D56, D68 to D57, D69 to D58, D70 to D59, D64 to D60, D65 to D61, D72 to D62, D73 to D63, D74 to D64, D75 to D65, D76 to D67, D77 to D68, D78 to D69, D79 to D70, D83 to D71, D84 to D72, D85 to D73, D86 to D74, D87 to D75, D81 to D76, D82 to D77, D89 to D78, D90 to D79, D7 to D8, D94 to D80, D95 to D81, D96 to D82, D97 to D83, D98 to D84, D92 to D85, D93 to D86, D100 to D87, D101 to D88, D105 to D89, D8 to D9, D106 to D90, D107 to D91, D108 to D92, D109 to D93, D103 to D94, D104 to D95, D111 to D96, D112 to D97, D117 to D98, D118 to D99, SW11 to SW10, SW12 to SW11, SW13 to SW12, SW15 to SW13, SW16 to SW14, SW17 to SW15, SW18 to SW16, SW19 to SW17, SW21 to SW18, SW22 to SW19, SW23 to SW20, SW24 to SW21, SW25 to SW22, SW26 to SW23, SW27 to SW24, SW28 to SW25, SW29 to SW26, SW30 to SW27, SW31 to SW28, SW32 to SW29, SW33 to SW30, SW34 to SW31, SW36 to SW32, SW37 to SW33, SW38 to SW34, SW39 to SW35, SW40 to SW36, SW41 to SW37, SW43 to SW38, SW44 to SW39, SW45 to SW40, SW46 to SW41, SW47 to SW42, SW49 to SW43, SW50 to SW44, SW51 to SW45, SW52 to SW46, SW53 to SW47, SW55 to SW48, SW56 to SW49, SW57 to SW50, SW58 to SW51, SW59 to SW52, SW60 to SW53, SW61 to SW54, SW62 to SW55, SW63 to SW56, SW64 to SW57, SW65 to SW58, SW66 to SW59, SW67 to SW60, SW68 to SW61, SW70 to SW62, SW9 to SW8, SW10 to SW9
Connections:
- D10 pad 2: LED_DATA_L -> Net-(D10-DIN)
- D118 pad 2: Net-(D139-A) -> /Matrix_Right/ENC_SW
- D59 pad 2: Net-(D70-A) -> /Matrix_Left/ENC_SW
- D68 pad 4: Net-(D77-DOUT) -> unconnected-(D68-DOUT-Pad4)
- D69 pad 2: LED_DATA_R -> Net-(D66-DOUT)
- D9 pad 4: Net-(D11-DIN) (its old number) -> unconnected-(D9-DOUT-Pad4)
- SW32 pad C: ROW5_L -> GND
- SW62 pad C: ROW5_R -> GND
- U2 pad 15: ROW1_L -> /Control_Left/LCD_CS
- U2 pad 16: ROW2_L -> ROW1_L
- U2 pad 17: ROW3_L -> ROW2_L
- U2 pad 18: ROW4_L -> ROW3_L
- U2 pad 19: ROW5_L -> ENC_CW_L
- U2 pad 20: unconnected-(U2-P0.31_BAT-Pad20) -> ENC_CC_L
- U2 pad 22: /Control_Left/LCD_CS -> ROW5_L
- U2 pad 23: ROW6_L -> ROW4_L
- U4 pad 15: ROW1_R -> /Control_Right/LCD_CS
- U4 pad 16: ROW2_R -> ROW1_R
- U4 pad 17: ROW3_R -> ROW2_R
- U4 pad 18: ROW4_R -> ROW3_R
- U4 pad 19: ROW5_R -> ENC_CW_R
- U4 pad 20: unconnected-(U4-P0.31_BAT-Pad20) -> ENC_CC_R
- U4 pad 22: /Control_Right/LCD_CS -> ROW5_R
- U4 pad 23: ROW6_R -> ROW4_R
