File: Hardware/ValkiriaSplit.kicad_pcb (KiCad board)
At the start: 2 copper layers, 285.5 x 93.5 mm, 266 parts, among them J1 BAT, J2 JTAG, J3 1.08_MIP_MODULE, J4 BAT, J5 JTAG, J6 1.08_MIP_MODULE, Q1 AO3401A, Q2 AO3401A, SW1 MSK12C02, SW10 PG1350, SW11 PG1350, SW12 PG1350, SW13 PG1350, SW14 PG1350, SW15 PG1350, SW16 PG1350, SW17 PG1350, SW18 PG1350, SW19 PG1350, SW2 SW_Push, SW20 PG1350, SW21 PG1350, SW22 PG1350, SW23 PG1350, SW24 PG1350, SW25 PG1350, SW26 PG1350, SW27 PG1350, SW28 PG1350, SW29 ENCODER, SW3 MSK12C02, SW30 PG1350, SW31 PG1350, SW32 PG1350, SW33 PG1350, SW34 PG1350, SW35 PG1350, SW36 PG1350, SW37 PG1350, SW38 PG1350, SW39 PG1350, SW4 SW_Push, SW40 PG1350, SW41 PG1350, SW42 PG1350, SW43 PG1350, SW44 PG1350, SW45 PG1350, SW46 PG1350, SW47 PG1350, SW48 PG1350, SW49 PG1350, SW5 PG1350, SW50 PG1350, SW51 PG1350, SW52 PG1350, SW53 PG1350, SW54 ENCODER, SW6 PG1350, SW7 PG1350, SW8 PG1350, SW9 PG1350, U1 TPS61040DBV, U2 XIAO-NRF52840-PLUS, U3 TPS61040DBV, U4 XIAO-NRF52840-PLUS

Commit message: Matrix routing and data lines
Routed some of the lines for the switch matrix.
Routed the singal lines for the MIP display.
Need to check clearenaces and spacing between the SPI lines.
Parts:
- added C67: 100n, Capacitor_SMD:C_0603_1608Metric, B.Cu at (174.0, 130.2)
- added C68: 100n, Capacitor_SMD:C_0603_1608Metric, B.Cu at (208.6, 200.2)
- added R21: 0, Resistor_SMD:R_0603_1608Metric, B.Cu at (174.0, 124.4)
- added R22: 0, Resistor_SMD:R_0603_1608Metric, B.Cu at (203.5, 193.7)
- J1, J4: footprint Custom_Parts:JST_PH_1x02_P2.00MM_SMD_HOR -> Custom_Parts:JST_ZH_1x02_P1.50MM_SMD_HORIZONTAL
- SW2, SW4: value SW_Push -> SWITCH
- moved R18 94.7 mm to (176.0, 111.8), turned to -90 degrees
- moved R17 92.6 mm to (174.0, 111.8), turned to -90 degrees
- moved R3 91.6 mm to (190.9, 114.8), turned to 90 degrees
- moved C40 74.0 mm to (174.0, 128.4)
- moved C39 73.6 mm to (174.0, 126.4)
- moved J4 70.4 mm to (216.1, 133.8), turned to -90 degrees
- moved J1 70.0 mm to (183.2, 134.0), turned to 90 degrees
- moved Q1 63.3 mm to (175.2, 145.6), turned to -90 degrees
- moved L1 59.3 mm to (181.4, 146.0), turned to 0 degrees
- moved R2 59.3 mm to (172.0, 142.2), turned to 90 degrees
- moved R4 56.9 mm to (185.8, 151.8)
- moved R5 56.8 mm to (182.4, 153.6)
- moved D1 54.7 mm to (175.2, 142.2)
- moved D2 54.1 mm to (186.4, 147.4)
- moved U1 53.5 mm to (181.4, 150.8)
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Connections:
- SW29 pad S1: ENC_SW_R -> /Matrix_Left/ENC_SW
- SW54 pad S1: ENC_SW_R -> /Matrix_Right/ENC_SW
- U2 pad 15: COL1_L -> COL6_L
- U2 pad 16: COL2_L -> ROW1_L
- U2 pad 17: COL3_L -> ROW2_L
- U2 pad 18: COL4_L -> unconnected-(U2-P0.09_NFC1-Pad18)
- U2 pad 19: COL5_L -> COL2_L
- U2 pad 2: ROW1_L -> COL5_L
- U2 pad 20: unconnected-(U2-P0.31_BAT-Pad20) -> ROW4_L
- U2 pad 23: ENC_SW_R -> ENC_SW_L
- U2 pad 3: ROW2_L -> COL3_L
- U2 pad 4: ROW3_L -> COL1_L
- U2 pad 5: ROW4_L -> COL4_L
- U2 pad 6: COL6_L -> ROW3_L
Routing:
- net COL6_L: track 46.0 -> 180.2 mm, vias 0 -> 2
- net COL5_L: track 69.1 -> 181.3 mm, vias 0 -> 2
- net COL3_L: track 46.0 -> 114.2 mm, vias 0 -> 2
- net ROW2_L: track 152.6 -> 209.6 mm, vias 6 -> 7
- net VBUSL: track 0.00 -> 53.6 mm
- net ROW1_L: track 152.6 -> 199.4 mm, vias 6 -> 7
- net VBATL: track 26.8 -> 54.2 mm
- net Net-(U2-P1.13_SCK): track 0.00 -> 12.6 mm
- net /Control_Left/MIP_SCK: track 0.00 -> 12.3 mm, vias 0 -> 2
- net Net-(U2-P1.15_MOSI): track 30.8 -> 21.0 mm
- net VREGL: track 0.00 -> 8.78 mm
- net COL1_L: track 42.1 -> 49.9 mm, vias 0 -> 1
- net /Control_Left/LED_EN: track 0.00 -> 6.85 mm
- net Net-(U2-P1.14_MISO): track 25.6 -> 18.8 mm
- net ENC_CC_L: track 0.00 -> 6.74 mm
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- added copper zone on B.Cu, net /Control_Left/VFB
- added copper zone on B.Cu, net /Control_Left/VSW
- added copper zone on B.Cu, net 5VL
- added copper zone on B.Cu, net VBUSL
- added copper zone on B.Cu, net VREGL
Other:
- outline, holes or cut-outs redrawn
